File: BoardRZA1.sch (KiCad schematic (older format))
At the start: 83 parts, among them CON1 USB-MINI-B, CON2 USB-MINI-B, P1 CONN_5X2, U1 RZ-A1L, U2 OSC_4PIN, U3 OSC_4PIN, U4 N25QXXX, U5 AS4C16M16S, X1 32.768k

Commit message: Ruteo de power. Reogranizado de la plaqueta y planos de masa
Parts:
- added C46, C53: 1u, SMD_Packages:SM0805, symbol Csmall
- added C47, C48, C49, C50: 1u, Capacitors_SMD:c_0805, symbol Csmall
- added C52: 100n, SMD_Packages:SM0805, symbol Csmall
- added CON4: BARREL_JACK, Connect:BARREL_JACK, symbol BARREL_JACK
- added R17: 1K, SMD_Packages:SM0805, symbol R
- added R18: 2K1, SMD_Packages:SM0805, symbol R
- added R20: 10k, SMD_Packages:SM0805, symbol R
- added SW1: RESET, Discret:SW_PUSH-12mm, symbol SW_PUSH
- added U6: BA3259HFP, Rohm:Rohm-HRP5, symbol BA3259HFP
- added U7: BU42xx, Rohm:SSOP-5, symbol BU42xx
- CON3: renamed from CON?; footprint (none) -> microsd:microSD
- gave numbers to parts that had none: 2
Connections:
- net +1.2V: now also C50.1, R17.1, U6.4 (Vo2)
- net +3.3V: now also C46.1, R20.2, U6.5 (Vo1), U7.2 (Vdd)
- net RESET: now also C53.2, R20.1, SW1.1, U7.1 (Vout)
- net VSS: now also C46.2, C47.2, C48.2, C49.2, C50.2, C52.2, C53.1, CON4.2, CON4.3, R18.1, SW1.2, U6.3 (GND), U6.FIN (GND), U7.3 (GND)
- net ET_MDC: now reaches U1.188 (P4_0/A17/VIO_VD/TIOC1B/ET_MDC/CTS1)
- net ET_MDIO: now reaches U1.189 (P4_1/A18/VIO_HD/TIOC2B/ET_MDIO/RTS1)
- net ET_TXD0: now reaches U1.192 (P8_0/LCD0_DATA0/ET_TXD0/SSISCK1/SCK3)
- net ET_TXD1: now reaches U1.194 (P8_1/LCD0_DATA1/ET_TXD1/SSIWS1/RxD3)
- net ET_TXD2: now reaches U1.198 (P8_2/LCD0_DATA2/ET_TXD2/SSITxD1/TxD3)
- net ET_TXD3: now reaches U1.199 (P8_3/LCD0_DATA3/ET_TXD3/SSIRxD1)
- net ET_TXCLK: now reaches U1.200 (P8_4/LCD0_DATA4/ET_TXCLK/CTS2/TIOC0A)
- net TX_TXER: now reaches U1.201 (P8_5/LCD0_DATA5/ET_TXER/RTS2/TIOC0B)
- net ET_COL: now reaches U1.70 (P8_14/LCD0_TCON6/ET_COL/SD_CD_0/SCK1)
- net ET_CRS: now reaches U1.71 (P8_15/ET_CRS/SD_WP_0/RxD1)
- new net: C47.1, C48.1, C49.1, CON4.1, U6.1 (Vcc)
- new net: R17.2, R18.2, U6.2 (ADJ)
- new net: C52.1, U7.5 (CT)

Commit message: Add ETH Add reset system Correct clock footprint Finish main routing and power/gnd planes
Parts:
- added C54, C63: 22u, SMD_Packages:SM0805, symbol Csmall
- added C55, C56, C57, C59, C60, C61, C62, C64, C65: 100n, SMD_Packages:SM0805, symbol Csmall
- added C58: 100p, SMD_Packages:SM0805, symbol Csmall
- added C66, C67: 22p, SMD_Packages:SM0805, symbol Csmall
- added J1: HR911105A, RJ45:RJ45_Pulse_J403-A, symbol HR911105A
- added L10: BLM18PG600, SMD_Packages:SM0805, symbol INDUCTOR_SMALL
- added R21: 6.49k, SMD_Packages:SM0805, symbol R
- added R22, R33, R34, R35: 4K7, SMD_Packages:SM0805, symbol R
- added R23, R24, R25, R26, R27, R28, R29, R30, R31, R32: 33R, SMD_Packages:SM0805, symbol R
- added R36, R37: 220R, SMD_Packages:SM0805, symbol R
- added R38, R39, R40, R41: 49.9, SMD_Packages:SM0805, symbol R
- added U8: KSZ8041MLL, smd_qfp:LQFP48-M05, symbol KSZ8041MLL
- added X2: 20MHz, Crystals:Crystal_HC49-SD_SMD, symbol CRYSTAL
- SW1: footprint Discret:SW_PUSH-12mm -> PushButton:RigthAnglePush
- U2: footprint OSC_4PIN:OSC_4PIN -> OSC_4PIN:OSC_2x2p5
Connections:
- net +3.3V: now also C54.1, C55.1, C56.1, C57.1, C59.1, L10.2, R22.1, R33.1, R34.2, R36.2, R37.1, U8.25 (VDDIO_3.3), U8.26 (VDDIO_3.3), U8.7 (VDDA_3.3), U8.8 (VDDA_3.3)
- net ET_COL: now also R24.1
- net ET_CRS: now also R23.1
- net ET_MDC: now also U1.72 (P9_0/ET_MDC/SD_D1_0/TxD1), U8.19 (MDC); no longer U1.188 (P4_0/A17/VIO_VD/TIOC1B/ET_MDC/CTS1)
- net ET_MDIO: now also U1.73 (P9_1/ET_MDIO/SD_D0_0/CTS0), R33.2, U8.18 (MDIO); no longer U1.189 (P4_1/A18/VIO_HD/TIOC2B/ET_MDIO/RTS1)
- net ET_TXCLK: now also R25.1
- net ET_TXD0: now also U8.35 (TXD0)
- net ET_TXD1: now also U8.36 (TXD1)
- net ET_TXD2: now also U8.38 (TXD2)
- net ET_TXD3: now also U8.39 (TXD3)
- net VSS: now also C54.2, C55.2, C56.2, C57.2, C58.2, C59.2, C60.2, C61.2, C62.2, C63.2, C64.2, C65.2, C66.2, C67.2, J1.13 (SHIELD), J1.14 (SHIELD), J1.8 (CHS_GND), R21.1, R35.1, U8.1 (GND), U8.13 (GND), U8.17 (GND), U8.2 (GND), U8.24 (GND), U8.3 (GND), U8.30 (GND), U8.37 (GND)
- net ET_RXCLK: now reaches U1.127 (P9_2/RSPCK2/ET_RXCLK/SD_CLK_0/RTS0/TIOC1A)
- net ET_RXCLK: now also R26.1
- net ET_RXER: now reaches U1.129 (P9_3/SSL20/ET_RXER/SD_CMD_0/SCK0/TIOC1B)
- net ET_RXER: now also R27.1
- net ET_RXDV: now reaches U1.135 (P9_4/MOSI2/ET_RXDV/SD_D3_0/RxD0/TIOC2A)
- net ET_RXDV: now also R28.1
- net ET_TXEN: now reaches U1.27 (P8_6/LCD0_DATA6/ET_TXEN/IRQ6/CTS1/TIOC0C)
- net ET_TXEN: now also U8.34 (TXEN)
- net ET_RXD0: now reaches U1.28 (P8_7/LCD0_DATA7/ET_RXD0/IRQ7/RTS1/TIOC0D)
- net ET_RXD0: now also R29.1
- net ET_RXD1: now reaches U1.29 (P8_8/LCD0_TCON0/ET_RXD1/AUDIO_XOUT/SCK2/AUDIO_XOUT3)
- net ET_RXD1: now also R30.1
- net ET_RXD2: now reaches U1.30 (P8_9/LCD0_TCON1/ET_RXD2/CAN1TX/RxD2/AUDIO_XOUT2)
- net ET_RXD2: now also R31.1
- net ET_RXD3: now reaches U1.35 (P8_10/LCD0_TCON2/ET_RXD3/CAN1RX/TxD2)
- net ET_RXD3: now also R32.1
- new net: J1.3 (RD+), R40.2, U8.10 (RX+)
- new net: J1.2 (TD-), R39.2, U8.11 (TX-)
- new net: J1.1 (TD+), R38.2, U8.12 (TX+)
- new net: C66.1, U8.14 (XO), X2.1
- new net: C67.1, U8.15 (XI), X2.2
- new net: C58.1, R21.2, U8.16 (REXT)
- new net: R32.2, U8.20 (RXD3/PHYAD0)
- new net: R31.2, U8.21 (RXD2/PHYAD1)
- new net: R30.2, U8.22 (RXD1/PHYAD2)
- new net: R29.2, U8.23 (RXD0/DUPLEX)
- new net: R28.2, U8.27 (RXDV/CONFIG2)
- new net: R26.2, U8.28 (RXCK)
- new net: R27.2, U8.29 (RXER/ISO)
- new net: R22.2, U8.32 (INTRP)
- new net: R25.2, U8.33 (TXCK)
- new net: R24.2, U8.40 (COL/CONFIG0)
- new net: R23.2, U8.41 (CRS/CONFIG1)
- new net: J1.6 (RD-), R41.2, U8.9 (RX-)
- new net: J1.12 (LEDY_A), R37.2
- new net: J1.4 (TCT), J1.5 (RCT), L10.1
- new net: J1.9 (LEDG_A), R36.1
- new net: C64.1, R38.1, R39.1
- new net: C65.1, R40.1, R41.1
- new net ET_1v8: C60.1, C61.1, C62.1, C63.1, U8.31 (VDD_1.8), U8.4 (VDDA_1.8), U8.5 (VDDA_1.8), U8.6 (V1.8_OUT)
- new net LED0: J1.10 (LEDG_K), R34.1, U8.42 (LED0/NWAYEN)
- new net LED1: J1.11 (LEDY_K), R35.2, U8.43 (LED1/SPEED)
- new net PHY_RESET: U8.47 (RST#)
- no-connect marks 9 -> 11
Other:
- note added: "LED0: PU\nLED1: PD"
- moved on the sheet: C38, C39, C40, C41, C42, C43, C44, C45, C46, C47, C48, C49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

Commit message: GPIO routed
Parts:
- added J2: SIL38, Pin_Headers:Pin_Header_Angled_1x38, symbol SIL38
- added R42: 10k, SMD_Packages:SM0805, symbol R
- added SW2: NMI, PushButton:RigthAnglePush, symbol SW_PUSH
Connections:
- net +3.3V: now also J2.1, R42.2
- net NMI: now also R42.1, SW2.1
- net VSS: now also J2.38, SW2.2
- net P1_14: now reaches U1.100 (P1_14/AN6/IRQ6/ET_RXD2/VIO_D6)
- net P1_14: now also J2.15
- net P1_15: now reaches U1.101 (P1_15/AN7/IRQ7/ET_RXD3/VIO_D7)
- net P1_15: now also J2.14
- net P1_0: now reaches U1.149 (P1_0/RIIC0SCL/IRQ4/ET_RXD0/DV0_DATA0)
- net P1_0: now also J2.13
- net P1_1: now reaches U1.150 (P1_1/RIIC0SDA/IRQ5/ET_RXD1/DV0_DATA1)
- net P1_1: now also J2.12
- net P1_2: now reaches U1.151 (P1_2/RIIC1SCL/IRQ6/ET_RXD2/DV0_DATA2)
- net P1_2: now also J2.11
- net P1_3: now reaches U1.152 (P1_3/RIIC1SDA/IRQ7/ET_RXD3/DV0_DATA3)
- net P1_3: now also J2.10
- net P1_4: now reaches U1.153 (P1_4/RIIC2SCL/IRQ0/DREQ0/VIO_D0)
- net P1_4: now also J2.9
- net P1_5: now reaches U1.154 (P1_5/RIIC2SDA/IRQ1/VIO_D1)
- net P1_5: now also J2.8
- net P1_6: now reaches U1.155 (P1_6/RIIC3SCL/IRQ2/SSIRxD0/VIO_D2)
- net P1_6: now also J2.7
- net P1_7: now reaches U1.156 (P1_7/RIIC3SDA/IRQ3/RxD2/VIO_D3)
- net P1_7: now also J2.6
- net P3_15: now reaches U1.157 (P3_15/A16/VIO_FLD/DV0_DATA15/TxD1)
- net P3_15: now also J2.5
- net P2_7: now reaches U1.159 (P2_7/CS0/SSISCK3/TIOC1A/IRQ2)
- net P2_7: now also J2.4
- net P2_8: now reaches U1.160 (P2_8/RD/SSITxD3/TIOC0A/CAN0TX)
- net P2_8: now also J2.3
- net P2_9: now reaches U1.161 (P2_9/A0/SSIWS3/SCK0/IRQ1/CAN0RX)
- net P2_9: now also J2.2
- net P6_6: now reaches U1.31 (P6_6/D22/LCD0_DATA14/SSITxD3/MLB_DAT)
- net P6_6: now also J2.37
- net P6_7: now reaches U1.32 (P6_7/D23/LCD0_DATA15/SSIRxD3/IRQ0/TIOC3A/RLIN30/RX)
- net P6_7: now also J2.36
- net P6_8: now reaches U1.33 (P6_8/D24/LCD0_DATA16/SSISCK0/IRQ1/TIOC3B/RLIN30/TX)
- net P6_8: now also J2.35
- net P8_11: now reaches U1.37 (P8_11/LCD0_TCON3/SSISCK2/SCK4)
- net P6_9: now reaches U1.38 (P6_9/D25/LCD0_DATA17/SSIWS0/IRQ2/TIOC3C)
- net P6_9: now also J2.34
- net P6_10: now reaches U1.40 (P6_10/D26/LCD0_DATA18/SSITxD0/IRQ3/TIOC3D/CAN1_TX)
- net P6_10: now also J2.33
- net P6_11: now reaches U1.41 (P6_11/D27/LCD0_DATA19/SSIRxD0/SSI_DATA2/SCK0/CAN1_RX)
- net P6_11: now also J2.32
- net P6_12: now reaches U1.43 (P6_12/D28/LCD0_DATA20/RSPCK1/SSI_SCK2/RTS0/DV0_DATA0)
- net P6_12: now also J2.31
- net P6_13: now reaches U1.46 (P6_13/D29/LCD0_DATA21/SSL10/SSI_WS2/CTS0/DV0_DATA1)
- net P6_13: now also J2.30
- net P6_14: now reaches U1.48 (P6_14/D30/LCD0_DATA22/MOSI1/SSI_DATA2/RxD0/DV0_DATA2)
- net P6_14: now also J2.29
- net P6_15: now reaches U1.49 (P6_15/D31/LCD0_DATA23/MISO1/TxD0/DV0_DATA3)
- net P6_15: now also J2.28
- net P7_8: now reaches U1.60 (P7_8/CS2/SSISCK1/DV0_CLK/IRQ3/TxD0)
- net P7_8: now also J2.27
- net P7_9: now reaches U1.61 (P7_9/A25/SSIWS1/DV0_VSYNC/IRQ5/SCK3/TIOC1A)
- net P7_9: now also J2.26
- net P7_10: now reaches U1.62 (P7_10/TEND0/SSITxD1/DV0_HSYNC/RxD3)
- net P7_10: now also J2.25
- net P7_11: now reaches U1.63 (P7_11/DACK0/SSIRxD1/CAN_CLK/SCK2/TxD3/AUDIO_XOUT/AUDIO_XOUT3)
- net P7_11: now also J2.24
- net P7_12: now reaches U1.64 (P8_12/LCD0_TCON4/SPDIF_IN/SSIWS2/RxD4)
- net P7_12: now also J2.23
- net P7_13: now reaches U1.66 (P8_13/LCD0_TCON5/SPDIF_OUT/SSI_DATA2/TxD4)
- net P7_13: now also J2.22
- net P1_8: now reaches U1.94 (P1_8/AN0/IRQ0/RxD0/DV0_DATA4)
- net P1_8: now also J2.21
- net P1_9: now reaches U1.95 (P1_9/AN1/IRQ1/RxD1/DV0_DATA5)
- net P1_9: now also J2.20
- net P1_10: now reaches U1.96 (P1_10/AN2/IRQ2/RxD2/DV0_DATA6)
- net P1_10: now also J2.19
- net P1_11: now reaches U1.97 (P1_11/AN3/IRQ3/RxD3/DV0_DATA7)
- net P1_11: now also J2.18
- net P1_12: now reaches U1.98 (P1_12/AN4/IRQ4/ET_RXD0/VIO_D4)
- net P1_12: now also J2.17
- net P1_13: now reaches U1.99 (P1_13/AN5/IRQ5/ET_RXD1/VIO_D5)
- net P1_13: now also J2.16
- no-connect marks 11 -> 15
Changed lines of the file:
@@
 LIBS:KSZ8041MLL
 LIBS:hr911105a
+LIBS:sil40
 LIBS:BoardRZA1-cache
 EELAYER 24 0
@@
 	16500 3900 16800 3900
 Wire Wire Line
-	16800 3700 16800 4000
+	16800 3050 16800 4000
 Wire Wire Line
 	16800 3700 16700 3700
@@
 Wire Wire Line
 	18500 24650 18500 24750
+$Comp
+L VSS #PWR063
+U 1 1 546806AB
+P 8350 12150
+F 0 "#PWR063" H 8350 12150 30  0001 C CNN
+F 1 "VSS" H 8350 12080 30  0000 C CNN
+F 2 "" H 8350 12150 60  0000 C CNN
+F 3 "" H 8350 12150 60  0000 C CNN
+	1    8350 12150
+	1    0    0    -1
+$EndComp
+Wire Wire Line
+	8350 12150 8350 11950
+Wire Wire Line
+	8350 11950 8100 11950
+$Comp
+L +3.3V #PWR064
+U 1 1 54681794
+P 8200 8100
+F 0 "#PWR064" H 8200 8060 30  0001 C CNN
+F 1 "+3.3V" H 8200 8210 30  0000 C CNN
+F 2 "" H 8200 8100 60  0000 C CNN
+F 3 "" H 8200 8100 60  0000 C CNN
+	1    8200 8100
+	1    0    0    -1
+$EndComp
+Wire Wire Line
+	8200 8100 8200 8250
+Wire Wire Line
+	8200 8250 8100 8250
+$Comp
+L SIL38 J2
+U 1 1 5468523A
+P 7650 10200
+F 0 "J2" H 7650 10150 60  0000 C CNN
+F 1 "SIL38" H 7650 10250 60  0000 C CNN
+F 2 "Pin_Headers:Pin_Header_Angled_1x38" H 7650 10200 60  0001 C CNN
+F 3 "" H 7650 10200 60  0000 C CNN
+	1    7650 10200
+	-1   0    0    -1
+$EndComp
+Text Label 27950 13350 0    60   ~ 0
+P1_0
+Text Label 27950 13250 0    60   ~ 0
+P1_1
+Text Label 27950 13150 0    60   ~ 0
+P1_2
+Text Label 27950 13050 0    60   ~ 0
+P1_3
+Text Label 27950 12950 0    60   ~ 0
+P1_4
+Text Label 27950 12850 0    60   ~ 0
+P1_5
+Text Label 27950 12750 0    60   ~ 0
+P1_6
+Text Label 27950 12650 0    60   ~ 0
+P1_7
+Text Label 8100 9450 0    60   ~ 0
+P1_0
+Text Label 8100 9350 0    60   ~ 0
+P1_1
+Text Label 8100 9250 0    60   ~ 0
+P1_2
+Text Label 8100 9150 0    60   ~ 0
+P1_3
+Text Label 8100 9050 0    60   ~ 0
+P1_4
+Text Label 8100 8950 0    60   ~ 0
+P1_5
+Text Label 8100 8850 0    60   ~ 0
+P1_6
+Text Label 8100 8750 0    60   ~ 0
+P1_7
+Text Label 27950 12550 0    60   ~ 0
+P3_15
+Text Label 27950 12350 0    60   ~ 0
+P2_7
+Text Label 27950 12250 0    60   ~ 0
+P2_8
+Text Label 27950 12150 0    60   ~ 0
+P2_9
+NoConn ~ 27950 11850
+Text Label 8100 8550 0    60   ~ 0
+P2_7
+Text Label 8100 8450 0    60   ~ 0
+P2_8
+Text Label 8100 8350 0    60   ~ 0
+P2_9
+Text Label 8100 8650 0    60   ~ 0
+P3_15
+Text Label 18650 17450 2    60   ~ 0
+P1_15
+Text Label 18650 17350 2    60   ~ 0
+P1_14
+Text Label 18650 17250 2    60   ~ 0
+P1_13
+Text Label 18650 17150 2    60   ~ 0
+P1_12
+Text Label 18650 17050 2    60   ~ 0
+P1_11
+Text Label 18650 16950 2    60   ~ 0
+P1_10
+Text Label 18650 16850 2    60   ~ 0
+P1_9
+Text Label 18650 16750 2    60   ~ 0
+P1_8
+Text Label 8100 9550 0    60   ~ 0
+P1_15
+Text Label 8100 9650 0    60   ~ 0
+P1_14
+Text Label 8100 9750 0    60   ~ 0
+P1_13
+Text Label 8100 9850 0    60   ~ 0
+P1_12
+Text Label 8100 9950 0    60   ~ 0
+P1_11
+Text Label 8100 10050 0    60   ~ 0
+P1_10
+Text Label 8100 10150 0    60   ~ 0
+P1_9
+Text Label 8100 10250 0    60   ~ 0
+P1_8
+$Comp
+L SW_PUSH SW2
+U 1 1 5468BE53
+P 16400 3050
+F 0 "SW2" H 16550 3160 50  0000 C CNN
+F 1 "NMI" H 16400 2970 50  0000 C CNN
+F 2 "PushButton:RigthAnglePush" H 16400 3050 60  0001 C CNN
+F 3 "" H 16400 3050 60  0000 C CNN
+	1    16400 3050
+	1    0    0    -1
+$EndComp
+$Comp
+L R R42
+U 1 1 5468BF93
+P 15600 3050
+F 0 "R42" V 15680 3050 40  0000 C CNN
+F 1 "10k" V 15607 3051 40  0000 C CNN
+F 2 "SMD_Packages:SM0805" V 15530 3050 30  0001 C CNN
+F 3 "" H 15600 3050 30  0000 C CNN
+	1    15600 3050
+	0    1    1    0
+$EndComp
+$Comp
+L +3.3V #PWR065
+U 1 1 5468C052
+P 15250 3050
+F 0 "#PWR065" H 15250 3010 30  0001 C CNN
+F 1 "+3.3V" H 15250 3160 30  0000 C CNN
+F 2 "" H 15250 3050 60  0000 C CNN
+F 3 "" H 15250 3050 60  0000 C CNN
+	1    15250 3050
+	0    -1   -1   0
+$EndComp
+Wire Wire Line
+	15250 3050 15350 3050
+Wire Wire Line
+	15850 3050 16100 3050
+Wire Wire Line
+	16700 3050 16800 3050
+Connection ~ 16800 3700
+Text Label 16050 3050 2    60   ~ 0
+NMI
+Text Label 18650 14050 2    60   ~ 0
+P7_8
+Text Label 18650 14150 2    60   ~ 0
+P7_9
+Text Label 18650 14250 2    60   ~ 0
+P7_10
+Text Label 18650 14350 2    60   ~ 0
+P7_11
+Text Label 18650 14450 2    60   ~ 0
+P7_12
+Text Label 18650 14550 2    60   ~ 0
+P7_13
+Text Label 8100 10850 0    60   ~ 0
+P7_8
+Text Label 8100 10750 0    60   ~ 0
+P7_9
+Text Label 8100 10650 0    60   ~ 0
+P7_10
+Text Label 8100 10550 0    60   ~ 0
+P7_11
+Text Label 8100 10450 0    60   ~ 0
+P7_12
+Text Label 8100 10350 0    60   ~ 0
+P7_13
+Text Label 18650 11950 2    60   ~ 0
+P6_6
+Text Label 18650 12050 2    60   ~ 0
+P6_7
+Text Label 18650 12150 2    60   ~ 0
+P6_8
+Text Label 18650 12350 2    60   ~ 0
+P8_11
+Text Label 18650 12550 2    60   ~ 0
+P6_10
+Text Label 18650 12450 2    60   ~ 0
+P6_9
+Text Label 18650 12650 2    60   ~ 0
+P6_11
+Text Label 18650 12750 2    60   ~ 0
+P6_12
+Text Label 18650 12950 2    60   ~ 0
+P6_13
+Text Label 18650 13050 2    60   ~ 0
+P6_14
+Text Label 18650 13150 2    60   ~ 0
+P6_15
+Text Label 8100 11850 0    60   ~ 0
+P6_6
+Text Label 8100 11750 0    60   ~ 0
+P6_7
+Text Label 8100 11650 0    60   ~ 0
+P6_8
+Text Label 8100 11450 0    60   ~ 0
+P6_10
+Text Label 8100 11550 0    60   ~ 0
+P6_9
+Text Label 8100 11350 0    60   ~ 0
+P6_11
+Text Label 8100 11250 0    60   ~ 0
+P6_12
+Text Label 8100 11150 0    60   ~ 0
+P6_13
+Text Label 8100 11050 0    60   ~ 0
+P6_14
+Text Label 8100 10950 0    60   ~ 0
+P6_15
+NoConn ~ 27950 14150
+NoConn ~ 27950 10550
+NoConn ~ 27950 10650
 $EndSCHEMATC

Commit message: Leds&buttons rerout eth out
Parts:
- added D1, D2, D3, D4: LED, LEDs:LED-0805, symbol LED
- added R43, R44: 10k, SMD_Packages:SM0805, symbol R
- added R45, R46, R47, R48: 1k, SMD_Packages:SM0805, symbol R
- added SW3: SW0, PushButton:RigthAnglePush, symbol SW_PUSH
- added SW4: SW1, PushButton:RigthAnglePush, symbol SW_PUSH
Connections:
- net +3.3V: now also D1.2 (K), D2.2 (K), D3.2 (K), D4.2 (K), R43.2, R44.2
- net LED0: now also U1.17 (P6_0/D16/LCD0_DATA8/RSPCK0/TCLKA/WDTOVF), R45.1; no longer J1.10 (LEDG_K), R34.1, U8.42 (LED0/NWAYEN)
- net LED1: now also U1.19 (P6_1/D17/LCD0_DATA9/SSL00/TCLKB), R46.1; no longer J1.11 (LEDY_K), R35.2, U8.43 (LED1/SPEED)
- net VSS: now also SW3.2, SW4.2
- net LED2: now reaches U1.20 (P6_2/D18/LCD0_DATA10/MOSI0/TCLKC)
- net LED2: now also R47.1
- net LED3: now reaches U1.22 (P6_3/D19/LCD0_DATA11/MISO0/TCLKD)
- net LED3: now also R48.1
- net SW1: now reaches U1.24 (P6_4/D20/LCD0_DATA12/SSISCK3/MLB_CLK)
- net SW1: now also R44.1, SW4.1
- net SW0: now reaches U1.26 (P6_5/D21/LCD0_DATA13/SSIWS3/MLB_SIG)
- net SW0: now also R43.1, SW3.1
- new net: D1.1 (A), R45.2
- new net: D2.1 (A), R46.2
- new net: D3.1 (A), R47.2
- new net: D4.1 (A), R48.2
- new net ET_LED0: J1.10 (LEDG_K), R34.1, U8.42 (LED0/NWAYEN)
- new net ET_LED1: J1.11 (LEDY_K), R35.2, U8.43 (LED1/SPEED)
- no-connect marks 15 -> 13
