File: BoardRZA1.sch (KiCad schematic (older format))
At the start: 145 parts, among them CON1 USB-MINI-B, CON2 USB-A-PCB, CON3 microSD, CON4 BARREL_JACK, J1 VGA, J2 SUPP32, K1 CONN_3, P1 CONN_5X2, P10 CONN_1, P11 CONN_1, P12 CONN_1, P13 CONN_1, P14 CONN_1, P15 CONN_1, P16 CONN_1, P17 CONN_1, P2 CONN_1, P3 CONN_1, P4 CONN_1, P5 CONN_1, P6 CONN_1, P7 CONN_1, P8 CONN_1, P9 CONN_1, SW1 RESET, SW2 NMI, SW3 SW0, SW4 SW1, U1 RZ-A1L, U2 13MHz, U3 48MHz, U4 N25QXXX, U5 AS4C16M16S, U6 NCP1117ST33T3G, U7 BU42xx, U8 ADV7125-lqfp48, U9 NCP1117ST12T3G, X1 32.768k

Commit message: Rework on minimize board
Signed-off-by: Martin Ribelotta <martinribelotta@gmail.com>
Parts:
- removed C54, C55, C56, C57, C58: 100n, Capacitors_SMD:C_0805, symbol Csmall
- removed CON4: BARREL_JACK, footprints:BARREL_JACK, symbol BARREL_JACK
- removed D5, D6: MBRA210, footprints:Diode-SMA_Standard, symbol DIODE
- removed J1: VGA, footprints:DB_15F-VGA, symbol VGA
- removed J2: SUPP32, Pin_Headers:Pin_Header_Angled_1x32, symbol SUPP32
- removed K1: CONN_3, Connect:SIL-3, symbol CONN_3
- removed P1: CONN_5X2, footprints:VASCH5x2, symbol CONN_5X2
- removed R21: 560R, Resistors_SMD:R_0805, symbol R
- removed R24, R25, R26: 75R, Resistors_SMD:R_0805, symbol R
- removed U8: ADV7125-lqfp48, w_smd_lqfp:lqfp48, symbol ADV7125-lqfp48
- added P1: CONN_02X04, Pin_Headers:Pin_Header_Straight_2x04, symbol CONN_02X04
- added P18, P19: CONN_01X40, Pin_Headers:Pin_Header_Straight_2x20, symbol CONN_01X40
- CON2: footprint footprints:USB_A -> Connect:USB_A_Vertical
Connections:
- net VBUS is gone; now on net +5v: CON1.1 (VBUS), U1.176 (VBUSIN0)
- net +3.3V: now also P18.3 (P3), P18.37 (P37), P18.38 (P38), P18.4 (P4), P19.3 (P3), P19.37 (P37), P19.38 (P38), P19.4 (P4)
- net JTAG_TCK: now also P1.2 (P2)
- net JTAG_TDI: now also P1.6 (P6)
- net JTAG_TDO: now also P1.4 (P4)
- net JTAG_TMS: now also P1.1 (P1)
- net JTAG_TRST: now also P1.8 (P8)
- net LCD_DATA0: now also P18.19 (P19)
- net LCD_DATA1: now also P18.20 (P20)
- net LCD_DATA10: now also P18.27 (P27)
- net LCD_DATA11: now also P18.28 (P28)
- net LCD_DATA12: now also P18.29 (P29)
- net LCD_DATA13: now also P18.30 (P30)
- net LCD_DATA14: now also P18.35 (P35)
- net LCD_DATA15: now also P18.36 (P36)
- net LCD_DATA16: now also P19.5 (P5)
- net LCD_DATA17: now also P19.8 (P8)
- net LCD_DATA18: now also P19.9 (P9)
- net LCD_DATA19: now also P19.10 (P10)
- net LCD_DATA2: now also P18.21 (P21)
- net LCD_DATA20: now also P19.11 (P11)
- net LCD_DATA21: now also P19.12 (P12)
- net LCD_DATA22: now also P19.13 (P13)
- net LCD_DATA23: now also P19.14 (P14)
- net LCD_DATA3: now also P18.22 (P22)
- net LCD_DATA4: now also P18.23 (P23)
- net LCD_DATA5: now also P18.24 (P24)
- net LCD_DATA6: now also P18.31 (P31)
- net LCD_DATA7: now also P18.32 (P32)
- net LCD_DATA8: now also P18.25 (P25)
- net LCD_DATA9: now also P18.26 (P26)
- net LCD_HSYNC: now also P18.33 (P33)
- net LCD_PCLK: now also P19.19 (P19)
- net LCD_VSYNC: now also P18.34 (P34)
- net LED0: now also P19.7 (P7)
- net LED1: now also P19.6 (P6)
- net LED2: now also P19.15 (P15)
- net LED3: now also P19.16 (P16)
- net LED4: now also P19.17 (P17)
- net NMI: now also P19.27 (P27)
- net P1_0: now also P18.5 (P5)
- net P1_1: now also P18.6 (P6)
- net P1_10: now also P19.31 (P31)
- net P1_11: now also P19.32 (P32)
- net P1_12: now also P19.33 (P33)
- net P1_13: now also P19.34 (P34)
- net P1_14: now also P19.35 (P35)
- net P1_15: now also P19.36 (P36)
- net P1_2: now also P18.7 (P7)
- net P1_3: now also P18.8 (P8)
- net P1_4: now also P18.9 (P9)
- net P1_5: now also P18.10 (P10)
- net P1_6: now also P18.11 (P11)
- net P1_7: now also P18.12 (P12)
- net P1_8: now also P19.29 (P29)
- net P1_9: now also P19.30 (P30)
- net P2_7: now also P18.14 (P14)
- net P2_8: now also P18.15 (P15)
- net P2_9: now also P18.16 (P16)
- net P3_15: now also P18.13 (P13)
- net P7_10: now also P19.25 (P25)
- net P7_11: now also P19.26 (P26)
- net P7_3: now also P19.18 (P18)
- net P7_5: now also P19.20 (P20)
- net P7_6: now also P19.21 (P21)
- net P7_7: now also P19.22 (P22)
- net P7_8: now also P19.23 (P23)
- net P7_9: now also P19.24 (P24)
- net P8_12(RXD): now also P1.3 (P3)
- net P8_13(TXD): now also P1.5 (P5)
- net RESET: now also P19.28 (P28)
- net SW0: now also P18.17 (P17)
- net SW1: now also P18.18 (P18)
- net VSS: now also P1.7 (P7), P18.1 (P1), P18.2 (P2), P18.39 (P39), P18.40 (P40), P19.1 (P1), P19.2 (P2), P19.39 (P39), P19.40 (P40)
- no-connect marks 14 -> 9
